File: Production Files/Logic_Level_Bidirectional-GiantPanel-v01.brd (EAGLE design)
At the start: 247.4 x 238.3 mm, 4044 parts, among them Q1 BSS138, Q10 BSS138, Q100 BSS138, Q101 BSS138, Q102 BSS138, Q103 BSS138, Q104 BSS138, Q105 BSS138, Q106 BSS138, Q107 BSS138, Q108 BSS138, Q109 BSS138, Q11 BSS138, Q110 BSS138, Q111 BSS138, Q112 BSS138, Q113 BSS138, Q114 BSS138, Q115 BSS138, Q116 BSS138, Q117 BSS138, Q118 BSS138, Q119 BSS138, Q12 BSS138, Q120 BSS138, Q121 BSS138, Q122 BSS138, Q123 BSS138, Q124 BSS138, Q125 BSS138, Q126 BSS138, Q127 BSS138, Q128 BSS138, Q129 BSS138, Q13 BSS138, Q130 BSS138, Q131 BSS138, Q132 BSS138, Q133 BSS138, Q134 BSS138, Q135 BSS138, Q136 BSS138, Q137 BSS138, Q138 BSS138, Q139 BSS138, Q14 BSS138, Q140 BSS138, Q141 BSS138, Q142 BSS138, Q143 BSS138, Q144 BSS138, Q145 BSS138, Q146 BSS138, Q147 BSS138, Q148 BSS138, Q149 BSS138, Q15 BSS138, Q150 BSS138, Q151 BSS138, Q152 BSS138, Q153 BSS138, Q154 BSS138, Q155 BSS138, Q156 BSS138, Q157 BSS138, Q158 BSS138, Q159 BSS138, Q16 BSS138, Q160 BSS138, Q161 BSS138, Q162 BSS138, Q163 BSS138, Q164 BSS138, Q165 BSS138, Q166 BSS138, Q167 BSS138, Q168 BSS138, Q169 BSS138, Q17 BSS138, Q170 BSS138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

Commit message: Recreated Panels both normal and Giant
Parts:
- moved E$9 1.05 mm to (4.57, 130.3)
- moved E$12 1.05 mm to (128.5, 130.3)
- moved E$1 1.05 mm to (4.57, 10.9)
- moved E$6 1.05 mm to (128.5, 10.9)
- moved E$10 0.13 mm to (243.0, 130.0)
- moved E$2 0.13 mm to (243.0, 10.7)
- moved E$4 0.13 mm to (119.0, 10.7)
- moved E$7 0.13 mm to (119.0, 130.0)
- moved E$5 0.13 mm to (119.0, 108.2)
- moved E$8 0.13 mm to (119.0, 227.6)
- moved E$11 0.13 mm to (243.0, 227.6)
- moved E$3 0.13 mm to (243.0, 108.2)
Other:
- outline, holes or cut-outs redrawn
